Commit message: 添加了轮子和小车的碰撞体积

File: learn03_robot_nav/src/robot_description/urdf/bot/actuator/caster.urdf.xacro (robot description, xacro)
@@ -1,36 +1,37 @@
 <?xml version="1.0"?>
 <robot xmlns:xacro="http://www.ros.org/wiki/xacro">
-    <xacro:macro name="camera_xacro" params="xyz">
-        <link name="camera_link">
+    <xacro:macro name="caster_xacro" params="caster_name xyz">
+        <!-- 机器人的IMU 惯性测量 -->
+        <link name="${caster_name}_link">
             <!-- 部件外观描述 -->
             <visual>
                 <!-- 沿自身几何中心偏移和旋转 -->
-                <origin xyz="0.0 0.0 0.0" rpy="0.0 0.0 0.0"/>
+                <origin xyz="0.0 0.0 0.0" rpy="0 0.0 0.0"/>
                 <!-- 几何形状 -->
                 <geometry>
-                    <box size="0.02 0.10 0.02"/>
+                    <sphere radius="0.016"/>
                 </geometry>
                 <!-- 材质和颜色描述 -->
-                <material name="black">
-                    <color rgba="0.0 0.0 0.0 0.5"/>
+                <material name="yellow">
+                    <color rgba="1.0 1.0 0.0 0.8"/>
                 </material>
             </visual>
             <collision>
                 <!-- 沿自身几何中心偏移和旋转 -->
-                <origin xyz="0.0 0.0 0.0" rpy="0.0 0.0 0.0"/>
+                <origin xyz="0.0 0.0 0.0" rpy="0 0.0 0.0"/>
                 <!-- 几何形状 -->
                 <geometry>
-                    <box size="0.02 0.10 0.02"/>
+                    <sphere radius="0.016"/>
                 </geometry>
                 <!-- 材质和颜色描述 -->
-                <material name="black">
-                    <color rgba="0.0 0.0 0.0 0.5"/>
+                <material name="yellow">
+                    <color rgba="1.0 1.0 0.0 0.8"/>
                 </material>
             </collision>
         </link>
         <!-- 机器人的关节，用于组合机器人的部件 -->
-        <joint name="camera_joint" type="fixed">
+        <joint name="${caster_name}_joint" type="fixed">
             <parent link="base_link"/>
-            <child link="camera_link"/>
+            <child link="${caster_name}_link"/>
             <origin xyz="${xyz}" rpy="0.0 0.0 0.0"/>
         </joint>

File: learn03_robot_nav/src/robot_description/urdf/bot/actuator/wheel.urdf.xacro (robot description, xacro)
@@ -1,37 +1,39 @@
 <?xml version="1.0"?>
 <robot xmlns:xacro="http://www.ros.org/wiki/xacro">
-    <xacro:macro name="camera_xacro" params="xyz">
-        <link name="camera_link">
+    <xacro:macro name="wheel_xacro" params="whell_name xyz">
+        <!-- 机器人的IMU 惯性测量 -->
+        <link name="${whell_name}_link">
             <!-- 部件外观描述 -->
             <visual>
                 <!-- 沿自身几何中心偏移和旋转 -->
-                <origin xyz="0.0 0.0 0.0" rpy="0.0 0.0 0.0"/>
+                <origin xyz="0.0 0.0 0.0" rpy="1.57079 0.0 0.0"/>
                 <!-- 几何形状 -->
                 <geometry>
-                    <box size="0.02 0.10 0.02"/>
+                    <cylinder radius="0.032" length="0.04"/>
                 </geometry>
                 <!-- 材质和颜色描述 -->
-                <material name="black">
-                    <color rgba="0.0 0.0 0.0 0.5"/>
+                <material name="yellow">
+                    <color rgba="1.0 1.0 0.0 0.8"/>
                 </material>
             </visual>
             <collision>
                 <!-- 沿自身几何中心偏移和旋转 -->
-                <origin xyz="0.0 0.0 0.0" rpy="0.0 0.0 0.0"/>
+                <origin xyz="0.0 0.0 0.0" rpy="1.57079 0.0 0.0"/>
                 <!-- 几何形状 -->
                 <geometry>
-                    <box size="0.02 0.10 0.02"/>
+                    <cylinder radius="0.032" length="0.04"/>
                 </geometry>
                 <!-- 材质和颜色描述 -->
-                <material name="black">
-                    <color rgba="0.0 0.0 0.0 0.5"/>
+                <material name="yellow">
+                    <color rgba="1.0 1.0 0.0 0.8"/>
                 </material>
             </collision>
         </link>
         <!-- 机器人的关节，用于组合机器人的部件 -->
-        <joint name="camera_joint" type="fixed">
+        <joint name="${whell_name}_joint" type="continuous">
             <parent link="base_link"/>
-            <child link="camera_link"/>
+            <child link="${whell_name}_link"/>
             <origin xyz="${xyz}" rpy="0.0 0.0 0.0"/>
+            <axis xyz="0 1 0"/>
         </joint>
     </xacro:macro>

File: learn03_robot_nav/src/robot_description/urdf/bot/base.urdf.xacro (robot description, xacro)
@@ -2,4 +2,6 @@
 <robot xmlns:xacro="http://www.ros.org/wiki/xacro">
     <xacro:macro name="base_xacro" params="length radius">
+        <link name="base_footprint">
+        </link>
         <!-- 机器人身体部分 -->
         <link name="base_link">
@@ -18,5 +20,23 @@
                 </material>
             </visual>
+            <collision>
+                <!-- 沿自身几何中心偏移和旋转 -->
+                <origin xyz="0.0 0.0 0.0" rpy="0.0 0.0 0.0"/>
+                <!-- 几何形状 -->
+                <geometry>
+                    <!-- 圆柱体 -->
+                    <cylinder radius="${radius}" length="${length}"/>
+                </geometry>
+                <!-- 材质和颜色描述 -->
+                <material name="white">
+                    <color rgba="1.0 1.0 1.0 0.5"/>
+                </material>
+            </collision>
         </link>
+        <joint name="joint_name" type="fixed">
+            <origin xyz="0.0 0.0 ${length/2.0 + 0.032 - 0.001}" rpy="0.0 0.0 0.0"/>
+            <parent link="base_footprint"/>
+            <child link="base_link"/>
+        </joint>
     </xacro:macro>
 </robot>

File: learn03_robot_nav/src/robot_description/urdf/bot/bot.urdf.xacro (robot description, xacro)
@@ -6,7 +6,14 @@
 <xacro:include filename="$(find robot_description)/urdf/bot/sensor/laser.urdf.xacro" />
 <xacro:include filename="$(find robot_description)/urdf/bot/sensor/camera.urdf.xacro" />
+<!-- 执行器部分 -->
+<xacro:include filename="$(find robot_description)/urdf/bot/actuator/wheel.urdf.xacro" />
+<xacro:include filename="$(find robot_description)/urdf/bot/actuator/caster.urdf.xacro" />
 <xacro:base_xacro length="0.12" radius="0.10" />
 <xacro:imu_xacro xyz="0.0 0.0 0.02" />
 <xacro:camera_xacro xyz="0.10 0.0 0.075" />
 <xacro:laser_xacro xyz="0.0 0.0 0.10" />
+<xacro:wheel_xacro whell_name="left_wheel" xyz="0 0.10 -0.06" />
+<xacro:wheel_xacro whell_name="right_wheel" xyz="0 -0.100 -0.06" />
+<xacro:caster_xacro caster_name="front_wheel" xyz="0.08 0 -0.076" />
+<xacro:caster_xacro caster_name="back_wheel" xyz="-0.08 0 -0.076" />
 </robot>

File: learn03_robot_nav/src/robot_description/urdf/bot/sensor/imu.urdf.xacro (robot description, xacro)
@@ -17,4 +17,16 @@
                 </material>
             </visual>
+            <collision>
+                <!-- 沿自身几何中心偏移和旋转 -->
+                <origin xyz="0.0 0.0 0.0" rpy="0.0 0.0 0.0"/>
+                <!-- 几何形状 -->
+                <geometry>
+                    <box size="0.02 0.02 0.02"/>
+                </geometry>
+                <!-- 材质和颜色描述 -->
+                <material name="black">
+                    <color rgba="0.0 0.0 0.0 0.5"/>
+                </material>
+            </collision>
         </link>
         <!-- 机器人的关节，用于组合机器人的部件 -->

File: learn03_robot_nav/src/robot_description/urdf/bot/sensor/laser.urdf.xacro (robot description, xacro)
@@ -17,4 +17,16 @@
                 </material>
             </visual>
+            <collision>
+                <!-- 沿自身几何中心偏移和旋转 -->
+                <origin xyz="0.0 0.0 0.0" rpy="0.0 0.0 0.0"/>
+                <!-- 几何形状 -->
+                <geometry>
+                    <cylinder radius="0.01" length="0.10"/>
+                </geometry>
+                <!-- 材质和颜色描述 -->
+                <material name="black">
+                    <color rgba="0.0 0.0 0.0 1.0"/>
+                </material>
+            </collision>
         </link>
         <!-- 雷达 -->
@@ -33,4 +45,16 @@
                 </material>
             </visual>
+            <collision>
+                <!-- 沿自身几何中心偏移和旋转 -->
+                <origin xyz="0.0 0.0 0.0" rpy="0.0 0.0 0.0"/>
+                <!-- 几何形状 -->
+                <geometry>
+                    <cylinder radius="0.02" length="0.02"/>
+                </geometry>
+                <!-- 材质和颜色描述 -->
+                <material name="black">
+                    <color rgba="0.0 0.0 0.0 1.0"/>
+                </material>
+            </collision>
         </link>
         <!-- 机器人的关节，用于组合机器人的部件 -->

Commit message: 基本运动解算器+gazebo模型

File: learn03_robot_nav/src/robot_description/urdf/bot/actuator/caster.urdf.xacro (robot description, xacro)
@@ -38,4 +38,10 @@
             <origin xyz="${xyz}" rpy="0.0 0.0 0.0"/>
         </joint>
+        <gazebo reference="${caster_name}_link">
+            <mu1 value="0.0"/>
+            <mu2 value="0.0"/>
+            <kp value="1000000000.0"/>
+            <kd value="1.0"/>
+        </gazebo>
     </xacro:macro>
 </robot>

File: learn03_robot_nav/src/robot_description/urdf/bot/actuator/wheel.urdf.xacro (robot description, xacro)
@@ -39,4 +39,10 @@
             <axis xyz="0 1 0"/>
         </joint>
+        <gazebo reference="${whell_name}_link">
+            <mu1 value="20.0"/>
+            <mu2 value="20.0"/>
+            <kp value="1000000000.0"/>
+            <kd value="1.0"/>
+        </gazebo>
     </xacro:macro>
 </robot>

File: learn03_robot_nav/src/robot_description/urdf/bot/bot.urdf.xacro (robot description, xacro)
@@ -9,4 +9,7 @@
 <xacro:include filename="$(find robot_description)/urdf/bot/actuator/wheel.urdf.xacro" />
 <xacro:include filename="$(find robot_description)/urdf/bot/actuator/caster.urdf.xacro" />
+<!-- 插件 -->
+<xacro:include filename="$(find robot_description)/urdf/bot/plugins/gazebo_control_plugin.xacro" />
+<xacro:include filename="$(find robot_description)/urdf/bot/plugins/gazebo_sensor_plugin.xacro" />
 <xacro:base_xacro length="0.12" radius="0.10" />
 <xacro:imu_xacro xyz="0.0 0.0 0.02" />
@@ -17,3 +20,5 @@
 <xacro:caster_xacro caster_name="front_wheel" xyz="0.08 0 -0.076" />
 <xacro:caster_xacro caster_name="back_wheel" xyz="-0.08 0 -0.076" />
+<xacro:gazebo_control_plugin />
+<xacro:gazebo_sensor_plugin />
 </robot>

File: learn03_robot_nav/src/robot_description/urdf/bot/sensor/camera.urdf.xacro (robot description, xacro)
@@ -31,4 +31,6 @@
             <xacro:box_inertia m="0.1" w="0.02" h="0.10" d="0.02" />
         </link>
+        <link name="camera_optical_link">
+        </link>
         <!-- 机器人的关节，用于组合机器人的部件 -->
         <joint name="camera_joint" type="fixed">
@@ -37,4 +39,10 @@
             <origin xyz="${xyz}" rpy="0.0 0.0 0.0"/>
         </joint>
+        <!-- 机器人的关节，用于组合机器人的部件 -->
+        <joint name="camera_optical_joint" type="fixed">
+            <parent link="camera_link"/>
+            <child link="camera_optical_link"/>
+            <origin xyz="0 0 0" rpy="${-pi/2} 0.0 ${-pi/2}"/>
+        </joint>
     </xacro:macro>
 </robot>

File: learn03_robot_nav/src/robot_description/urdf/bot/sensor/laser.urdf.xacro (robot description, xacro)
@@ -72,4 +72,10 @@
             <origin xyz="${xyz}" rpy="0.0 0.0 0.0"/>
         </joint>
+        <gazebo reference="laser_cylinder_link">
+            <material>Gazebo/Black</material>
+        </gazebo>
+        <gazebo reference="laser_link">
+            <material>Gazebo/Black</material>
+        </gazebo>
     </xacro:macro>
 </robot>
